File: Hardware/Prototype/Prototype.kicad_sch (KiCad schematic)
At the start: 0 parts

Commit message: board
Parts:
- added Adafruit_Micro_SD: Conn_01x09, symbol Connector_Generic:Conn_01x09
- added BZ1: Buzzer, symbol Device:Buzzer
- added ESP32_devkit: Conn_02x22_Odd_Even, symbol Connector_Generic:Conn_02x22_Odd_Even
- added I2SMic(ICS43434), JI2SMic(ICS43434)_2: Conn_01x06, symbol Connector_Generic:Conn_01x06
- added OLED: Conn_01x04, symbol Connector_Generic:Conn_01x04
- added SW1: SW_SPST, symbol Switch:SW_SPST

Commit message: reviewed schematic
Parts:
- removed ESP32_devkit: Conn_02x22_Odd_Even, symbol Connector_Generic:Conn_02x22_Odd_Even
- added U1: ESP32-S3-WROOM-2, RF_Module:ESP32-S3-WROOM-2, symbol RF_Module:ESP32-S3-WROOM-2
Connections:
- new net: U1.1 (GND), U1.40 (GND), U1.41 (GND)
Other:
- moved on the sheet: JI2SMic(ICS43434)_2, OLED
Changed lines of the file:
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@@
 	(symbol
 		(lib_id "Connector_Generic:Conn_01x06")
-		(at 219.71 86.36 0)
+		(at 226.06 85.09 0)
 		(unit 1)
 		(exclude_from_sim no)
@@
 		(fields_autoplaced yes)
 		(property "Reference" "JI2SMic(ICS43434)_2"
-			(at 222.25 86.3599 0)
+			(at 228.6 85.0899 0)
 			(effects
 				(font
@@
 		)
 		(property "Value" "Conn_01x06"
-			(at 222.25 88.8999 0)
+			(at 228.6 87.6299 0)
 			(effects
 				(font
@@
 		)
 		(property "Footprint" ""
-			(at 219.71 86.36 0)
+			(at 226.06 85.09 0)
 			(effects
 				(font
@@
 		)
 		(property "Datasheet" "~"
-			(at 219.71 86.36 0)
+			(at 226.06 85.09 0)
 			(effects
 				(font
@@
 		)
 		(property "Description" "Generic connector, single row, 01x06, script generated (kicad-library-utils/schlib/autogen/connector/)"
-			(at 219.71 86.36 0)
+			(at 226.06 85.09 0)
 			(effects
 				(font
@@
 	)
 	(symbol
-		(lib_id "Connector_Generic:Conn_02x22_Odd_Even")
-		(at 101.6 118.11 0)
+		(lib_id "RF_Module:ESP32-S3-WROOM-2")
+		(at 114.3 109.22 0)
 		(unit 1)
 		(exclude_from_sim no)
@@
 		(dnp no)
 		(fields_autoplaced yes)
-		(property "Reference" "ESP32_devkit"
-			(at 102.87 86.36 0)
-			(effects
-				(font
-					(size 1.27 1.27)
-				)
-			)
-		)
-		(property "Value" "Conn_02x22_Odd_Even"
-			(at 102.87 88.9 0)
-			(effects
-				(font
-					(size 1.27 1.27)
-				)
-			)
-		)
-		(property "Footprint" ""
-			(at 101.6 118.11 0)
-			(effects
-				(font
-					(size 1.27 1.27)
-				)
-				(hide yes)
-			)
-		)
-		(property "Datasheet" "~"
-			(at 101.6 118.11 0)
-			(effects
-				(font
-					(size 1.27 1.27)
-				)
-				(hide yes)
-			)
-		)
-		(property "Description" "Generic connector, double row, 02x22, odd/even pin numbering scheme (row 1 odd numbers, row 2 even numbers), script generated (kicad-library-utils/schlib/autogen/connector/)"
-			(at 101.6 118.11 0)
-			(effects
-				(font
-					(size 1.27 1.27)
-				)
-				(hide yes)
-			)
+		(property "Reference" "U1"
+			(at 116.4433 58.42 0)
+			(effects
+				(font
+					(size 1.27 1.27)
+				)
+				(justify left)
+			)
+		)
+		(property "Value" "ESP32-S3-WROOM-2"
+			(at 116.4433 60.96 0)
+			(effects
+				(font
+					(size 1.27 1.27)
+				)
+				(justify left)
+			)
+		)
+		(property "Footprint" "RF_Module:ESP32-S3-WROOM-2"
+			(at 114.3 170.18 0)
+			(effects
+				(font
+					(size 1.27 1.27)
+				)
+				(hide yes)
+			)
+		)
+		(property "Datasheet" "https://www.espressif.com/sites/default/files/documentation/esp32-s3-wroom-2_datasheet_en.pdf"
+			(at 114.3 172.72 0)
+			(effects
+				(font
+					(size 1.27 1.27)
+				)
+				(hide yes)
+			)
+		)
+		(property "Description" "RF Module, 2.4 GHz, Wi­-Fi, Bluetooth, BLE, ESP32­-S3R8V"
+			(at 114.3 109.22 0)
+			(effects
+				(font
+					(size 1.27 1.27)
+				)
+				(hide yes)
+			)
+		)
+		(pin "40"
+		)
+		(pin "27"
+		)
+		(pin "39"
+		)
+		(pin "4"
+		)
+		(pin "15"
+		)
+		(pin "7"
+		)
+		(pin "12"
+		)
+		(pin "5"
+		)
+		(pin "19"
+		)
+		(pin "6"
+		)
+		(pin "20"
+		)
+		(pin "17"
+		)
+		(pin "8"
+		)
+		(pin "18"
+		)
+		(pin "9"
+		)
+		(pin "21"
+		)
+		(pin "13"
+		)
+		(pin "22"
+		)
+		(pin "14"
+		)
+		(pin "10"
+		)
+		(pin "32"
+		)
+		(pin "11"
+		)
+		(pin "23"
+		)
+		(pin "31"
+		)
+		(pin "38"
+		)
+		(pin "41"
+		)
+		(pin "29"
+		)
+		(pin "30"
 		)
 		(pin "3"
 		)
+		(pin "28"
+		)
 		(pin "1"
 		)
-		(pin "5"
-		)
-		(pin "7"
-		)
-		(pin "9"
-		)
-		(pin "11"
-		)
-		(pin "13"
-		)
-		(pin "15"
-		)
-		(pin "17"
-		)
-		(pin "19"
-		)
-		(pin "21"
-		)
-		(pin "23"
+		(pin "2"
+		)
+		(pin "26"
+		)
+		(pin "34"
+		)
+		(pin "36"
+		)
+		(pin "35"
+		)
+		(pin "24"
 		)
 		(pin "25"
 		)
-		(pin "27"
-		)
-		(pin "29"
-		)
-		(pin "31"
+		(pin "16"
 		)
 		(pin "33"
 		)
-		(pin "35"
-		)
 		(pin "37"
-		)
-		(pin "39"
-		)
-		(pin "41"
-		)
-		(pin "43"
-		)
-		(pin "2"
-		)
-		(pin "4"
-		)
-		(pin "6"
-		)
-		(pin "8"
-		)
-		(pin "10"
-		)
-		(pin "12"
-		)
-		(pin "14"
-		)
-		(pin "16"
-		)
-		(pin "18"
-		)
-		(pin "20"
-		)
-		(pin "22"
-		)
-		(pin "24"
-		)
-		(pin "26"
-		)
-		(pin "28"
-		)
-		(pin "30"
-		)
-		(pin "32"
-		)
-		(pin "34"
-		)
-		(pin "36"
-		)
-		(pin "38"
-		)
-		(pin "40"
-		)
-		(pin "42"
-		)
-		(pin "44"
 		)
 		(instances
 			(project ""
 				(path "/06300a21-1646-41b0-b473-1c39557d6dab"
-					(reference "ESP32_devkit")
+					(reference "U1")
 					(unit 1)
 				)
@@
 	(symbol
 		(lib_id "Connector_Generic:Conn_01x04")
-		(at 144.78 163.83 0)
+		(at 101.6 177.8 0)
 		(unit 1)
 		(exclude_from_sim no)
@@
 		(fields_autoplaced yes)
 		(property "Reference" "OLED"
-			(at 147.32 163.8299 0)
+			(at 104.14 177.7999 0)
 			(effects
 				(font
@@
 		)
 		(property "Value" "Conn_01x04"
-			(at 147.32 166.3699 0)
+			(at 104.14 180.3399 0)
 			(effects
 				(font
@@
 		)
 		(property "Footprint" ""
-			(at 144.78 163.83 0)
+			(at 101.6 177.8 0)
 			(effects
 				(font
@@
 		)
 		(property "Datasheet" "~"
-			(at 144.78 163.83 0)
+			(at 101.6 177.8 0)
 			(effects
 				(font
@@
 		)
 		(property "Description" "Generic connector, single row, 01x04, script generated (kicad-library-utils/schlib/autogen/connector/)"
-			(at 144.78 163.83 0)
-			(effects
-				(font
+			(at 101.6 177.8 0)
+			(effects
+				(font
