File: Hardware/Keyfob Board/Keyfob Board.kicad_sch (KiCad schematic)
At the start: 10 parts, among them SW1 SW_Push, SW2 SW_Push, SW3 SW_Push, SW4 SW_Push, U1 MDBT42Q-512K

Commit message: drafted contact mic pcb layout
Parts:
- TP1, TP2, TP3, TP4, TP5: footprint (none) -> TestPoint:TestPoint_THTPad_D1.5mm_Drill0.7mm
Connections:
- net -BATT: now also TP4.1
- no-connect marks 27 -> 29
Other:
- moved on the sheet: TP4
Changed lines of the file:
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@@
 		(color 0 0 0 0)
 	)
+	(junction
+		(at 147.32 110.49)
+		(diameter 0)
+		(color 0 0 0 0)
+	)
 	(no_connect
 		(at 167.64 85.09)
@@
 	)
 	(no_connect
+		(at 127 52.07)
+	)
+	(no_connect
 		(at 167.64 92.71)
+	)
+	(no_connect
+		(at 127 46.99)
 	)
 	(no_connect
@@
 			)
 		)
-		(property "Footprint" ""
+		(property "Footprint" "TestPoint:TestPoint_THTPad_D1.5mm_Drill0.7mm"
 			(at 127 80.01 0)
 			(effects
@@
 	(symbol
 		(lib_id "Connector:TestPoint")
-		(at 147.32 109.22 90)
+		(at 147.32 110.49 90)
 		(unit 1)
 		(exclude_from_sim no)
@@
 		(dnp no)
 		(property "Reference" "TP4"
-			(at 140.97 109.728 90)
+			(at 140.97 110.998 90)
 			(effects
 				(font
@@
 		)
 		(property "Value" "TestPoint"
-			(at 141.986 112.268 90)
-			(effects
-				(font
-					(size 1.27 1.27)
-				)
-				(hide yes)
-			)
-		)
-		(property "Footprint" ""
-			(at 147.32 104.14 0)
+			(at 141.986 113.538 90)
+			(effects
+				(font
+					(size 1.27 1.27)
+				)
+				(hide yes)
+			)
+		)
+		(property "Footprint" "TestPoint:TestPoint_THTPad_D1.5mm_Drill0.7mm"
+			(at 147.32 105.41 0)
 			(effects
 				(font
@@
 		)
 		(property "Datasheet" "~"
-			(at 147.32 104.14 0)
+			(at 147.32 105.41 0)
 			(effects
 				(font
@@
 		)
 		(property "Description" "test point"
-			(at 147.32 109.22 0)
+			(at 147.32 110.49 0)
 			(effects
 				(font
@@
 			)
 		)
-		(property "Footprint" ""
+		(property "Footprint" "TestPoint:TestPoint_THTPad_D1.5mm_Drill0.7mm"
 			(at 127 82.55 0)
 			(effects
@@
 			)
 		)
-		(property "Footprint" ""
+		(property "Footprint" "TestPoint:TestPoint_THTPad_D1.5mm_Drill0.7mm"
 			(at 149.86 34.29 0)
 			(effects
@@
 			)
 		)
-		(property "Footprint" ""
+		(property "Footprint" "TestPoint:TestPoint_THTPad_D1.5mm_Drill0.7mm"
 			(at 127 85.09 0)
 			(effects
