File: Hardware/Main Board/Adafruit OLED 128x32 Mono I2C STEMMA QT rev B/Adafruit OLED 128x32 Mono I2C STEMMA QT rev B.kicad_sch (KiCad schematic)
At the start: 27 parts, among them IC5 APX803, Q2 BSS138, U2 AP2112K-3.3

Commit message: drafted entire main board schematic and assigned footprints
Parts:
- renumbered C2 to C14, C3 to C15, C1 to C16, C6 to C17, C7 to C18, C8 to C19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
